Commit message: changed the prefix names so it doesnt overlap with the UR packages prefix names

File: mir_description/urdf/include/imu.gazebo.urdf.xacro (robot description, xacro)
@@ -1,6 +1,6 @@
 <?xml version="1.0"?>
 <robot xmlns:xacro="http://ros.org/wiki/xacro">
-  <xacro:arg name="tf_prefix" default="" />
-  <xacro:property name="prefix" value="$(arg tf_prefix)" />
+  <xacro:arg name="mir_prefix" default="" />
+  <xacro:property name="prefix" value="$(arg mir_prefix)" />
   <xacro:property name="imu_frame" value="${prefix + '/imu_frame' if prefix != '' else 'imu_frame'}" />
   <xacro:macro name="imu_gazebo" params="link imu_topic update_rate">

File: mir_description/urdf/mir.urdf.xacro (robot description, xacro)
@@ -2,6 +2,6 @@
 <robot xmlns:xacro="http://ros.org/wiki/xacro" name="mir">
   <xacro:include filename="$(find mir_description)/urdf/include/mir_v1.urdf.xacro" />
-  <xacro:arg name="tf_prefix" default="" />
-  <xacro:property name="prefix" value="$(arg tf_prefix)" />
+  <xacro:arg name="mir_prefix" default="" />
+  <xacro:property name="prefix" value="$(arg mir_prefix)" />
   <xacro:property name="prefix_with_slash" value="${prefix + '/' if prefix != '' else ''}" />
   <xacro:mir prefix="${prefix_with_slash}" />
